File: Hardware/DIP_REFLOW_v1.sch (EAGLE design)
At the start: 32 parts, among them IC1 7805, J1 ICSP, Q1 2N3904, Q2 2N3904, Q3 2N3904, U1 ATMEGA328P_PDIP, U2 LCD-16X2SILK, Y1 16Mhz

Commit message: Updates and Fixes
Parts:
- removed LOGO1: OSHW-LOGOL, SparkFun-Aesthetics:OSHW-LOGOL
Changed lines of the file:
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@@
 <part name="JP7" library="adafruit" deviceset="PINHD-1X6" device="" value="MAX31855"/>
 <part name="R6" library="SparkFun-Electromechanical" deviceset="TRIMPOT" device="-PTH-KNOB" value="10k Ohm"/>
-<part name="LOGO1" library="SparkFun-Aesthetics" deviceset="OSHW-LOGO" device="L"/>
 <part name="FRAME1" library="SparkFun-Aesthetics" deviceset="FRAME-LETTER" device=""/>
 </parts>
@@
 <instance part="JP7" gate="A" x="195.58" y="162.56" rot="R180"/>
 <instance part="R6" gate="R?" x="220.98" y="111.76"/>
-<instance part="LOGO1" gate="G$1" x="134.62" y="10.16"/>
 <instance part="FRAME1" gate="G$1" x="0" y="0"/>
 <instance part="FRAME1" gate="G$2" x="147.32" y="0"/>
